File: PiHAT_Test.kicad_pcb (KiCad board)
At the start: 2 copper layers, 24 parts, among them CN1 DYNAMIXEL XL-320 MOLEX-53253-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, CN2 DYNAMIXEL XL-320 MOLEX-53253-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, CN3 DYNAMIXEL XL-320 MOLEX-53253-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, CN4 DYNAMIXEL XL-320 MOLEX-53253-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, CN5 DYNAMIXEL XL-320 MOLEX-53253-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, CN6 DYNAMIXEL XL-320 MOLEX-53253-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, J1_I2C1 I2C_1, U1 LM7805_TO220, U2 Alimentation 12v

Commit message: Add 12V+ power and Gerber files
Routing:
- net +12V: track 108.2 -> 0.00 mm
- added copper zone on F.Cu, net +12V
Other:
- board outline added: 33 x 72 mm
