File: PiHAT_Test.kicad_pcb (KiCad board)
At the start: 2 copper layers, 33 x 72 mm, 24 parts, among them CN1 DYNAMIXEL XL-320 MOLEX-53253-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, CN2 DYNAMIXEL XL-320 MOLEX-53253-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, CN3 DYNAMIXEL XL-320 MOLEX-53253-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, CN4 DYNAMIXEL XL-320 MOLEX-53253-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, CN5 DYNAMIXEL XL-320 MOLEX-53253-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, CN6 DYNAMIXEL XL-320 MOLEX-53253-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, J1_I2C1 I2C_1, U1 LM7805_TO220, U2 Alimentation 12v

Commit message: Correct 5V regulator 12V input
Connections:
- H1 pad 9: GND -> unconnected-(H1-Pad9)
Routing:
- net +12V: track 0.00 -> 8.07 mm
- net GND: track 2.12 -> 1.52 mm
- net unconnected-(H1-Pad9): track 0.00 -> 0.61 mm
Changed lines of the file:
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@@
 	(net 40 "unconnected-(H1-Pad19)")
 	(net 41 "unconnected-(J1_I2C1-Pad5)")
+	(net 42 "unconnected-(H1-Pad9)")
 	(footprint "Module:Raspberry_Pi_Zero_Socketed_THT_FaceDown_MountingHoles"
 		(layer "F.Cu")
@@
 			(layers "*.Cu" "*.Mask")
 			(remove_unused_layers no)
-			(net 2 "GND")
+			(net 42 "unconnected-(H1-Pad9)")
 			(pinfunction "9")
 			(pintype "unspecified")
@@
 	)
 	(segment
-		(start 138.472182 119.987818)
-		(end 139 119.987818)
+		(start 138 78.5)
+		(end 139 77.5)
 		(width 0.4)
-		(layer "B.Cu")
-		(net 2)
+		(layer "F.Cu")
+		(net 1)
 	)
 	(segment
-		(start 127.87 82.63)
-		(end 128 82.5)
-		(width 0.2)
-		(layer "B.Cu")
-		(net 2)
+		(start 139 77.5)
+		(end 139 76.5)
+		(width 0.4)
+		(layer "F.Cu")
+		(net 1)
 	)
 	(segment
-		(start 138.012182 119.987818)
-		(end 139 119.987818)
-		(width 0.2)
-		(layer "B.Cu")
-		(net 2)
+		(start 136 78.5)
+		(end 138 78.5)
+		(width 0.4)
+		(layer "F.Cu")
+		(net 1)
 	)
 	(segment
-		(start 127.87 82.87)
-		(end 128 83)
-		(width 0.2)
-		(layer "B.Cu")
-		(net 2)
+		(start 134.54 77.04)
+		(end 136 78.5)
+		(width 0.4)
+		(layer "F.Cu")
+		(net 1)
 	)
 	(segment
-		(start 127.87 82.74)
-		(end 127.87 82.87)
-		(width 0.2)
+		(start 132.95 77.04)
+		(end 134.54 77.04)
+		(width 0.4)
+		(layer "F.Cu")
+		(net 1)
+	)
+	(segment
+		(start 138.472182 119.987818)
+		(end 139 119.987818)
+		(width 0.4)
 		(layer "B.Cu")
 		(net 2)
 	)
 	(segment
-		(start 127.87 82.74)
-		(end 127.87 82.63)
+		(start 138.012182 119.987818)
+		(end 139 119.987818)
 		(width 0.2)
 		(layer "B.Cu")
@@
 		(net 31)
 	)
+	(segment
+		(start 127.87 82.63)
+		(end 128 82.5)
+		(width 0.2)
+		(layer "B.Cu")
+		(net 42)
+	)
+	(segment
+		(start 127.87 82.87)
+		(end 128 83)
+		(width 0.2)
+		(layer "B.Cu")
+		(net 42)
+	)
+	(segment
+		(start 127.87 82.74)
+		(end 127.87 82.87)
+		(width 0.2)
+		(layer "B.Cu")
+		(net 42)
+	)
+	(segment
+		(start 127.87 82.74)
+		(end 127.87 82.63)
+		(width 0.2)
+		(layer "B.Cu")
+		(net 42)
+	)
 	(zone
